File: PCB/MQTTDecoderExpansionBoard.kicad_pcb (KiCad board)
At the start: 2 copper layers, 55.9 x 91.4 mm, 21 parts, among them J1 Conn_01x08_Female, J10 Conn_01x16_Female, J11 Conn_01x20_Female, J12 Conn_01x03_Female, J2 Conn_01x16_Female, J3 Conn_01x08_Female, J4 Conn_01x16_Female, J5 Conn_01x16_Female, J6 Conn_01x16_Female, J7 Conn_01x20_Female, J8 Conn_01x16_Female, J9 Conn_01x16_Female, U2 LM317_TO-220

Commit message: fixed up files
Parts:
- R1, R2: footprint Resistor_THT:R_Axial_DIN0204_L3.6mm_D1.6mm_P7.62mm_Horizontal -> Resistor_THT:R_Axial_DIN0207_L6.3mm_D2.5mm_P10.16mm_Horizontal
- moved R1 3.81 mm to (165.1, 121.9)
- moved R2 1.27 mm to (154.9, 116.8)
Routing:
- net Net-(J10-Pad1): track 250.8 -> 249.2 mm
- net Net-(J9-Pad1): track 229.0 -> 230.5 mm
- net Net-(R1-Pad2): track 20.8 -> 21.4 mm
Other:
- board text added: "TrainNode v0.1 JMRI MQTT I/O Controller Rewind2B4"
- board text removed: "TrainNode JMRI MQTT I/O Controller Rewind2B4"
